File: EduboardV2_ESP32/Debugger_FT2232HL.kicad_sch (KiCad schematic)
At the start: 63 parts, among them Q1 S8050_C139514, Q2 S8050_C139514, Q3 AO3401A, U2 FT2232HL, U3 M93C46-WMN6TP, U5 LD1117S33TR_SOT223, Y2 12MHz

Commit message: finalize Data. Add Logo and Text
Parts:
- C1, C2: JLCPCB Part # (none) -> C123529; LCSC Part (none) -> C123529
- C10, C11, C12, C13, C14, C15, C16, C26, C28, C3, C8, C9: JLCPCB Part # (none) -> C105907; LCSC Part (none) -> C105907
- C25, C27, C4, C5, C6, C7: JLCPCB Part # (none) -> C76642; LCSC Part (none) -> C76642
- JP1, JP2, JP3, JP4: now left out of the parts list
- R1, R13, R14, R25: JLCPCB Part # (none) -> C115003; LCSC Part (none) -> C115003
- R10, R11, R12: JLCPCB Part # (none) -> C657300; LCSC Part (none) -> C657300
- R15, R16, R21, R29, R30, R31, R32, R5: JLCPCB Part # (none) -> C465460; LCSC Part (none) -> C465460
- R17, R18, R2, R3, R4, R6, R7: JLCPCB Part # (none) -> C116677; LCSC Part (none) -> C116677
- R8: JLCPCB Part # (none) -> C217840; LCSC Part (none) -> C217840
- R9: JLCPCB Part # (none) -> C203265; LCSC Part (none) -> C203265
- Y2: LCSC Part (none) -> C93114
Connections:
- net D_N: now reaches R29.2, R31.2, U2.7 (DM)
- net D_P: now reaches R30.2, R32.2, U2.8 (DP)
