File: EduboardV2_ESP32/EduboardV2_ESP32.kicad_sch (KiCad schematic)
At the start: 17 parts, among them J1 EduboardV2 PCIE UP Board Conn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, SW1 K2-1102SP-C4SC-04, SW2 K2-1102SP-C4SC-04, U1 ESP32-WROOM-E

Commit message: finalize Data. Add Logo and Text
Parts:
- C2: JLCPCB Part # (none) -> C105907; LCSC Part (none) -> C105907
- C2: JLCPCB Part # (none) -> C128624; LCSC Part (none) -> C128624
- J1, JP7, JP8: now left out of the parts list
- R13: JLCPCB Part # (none) -> C115003; LCSC Part (none) -> C115003
- R17: JLCPCB Part # (none) -> C116677; LCSC Part (none) -> C116677
Changed lines of the file:
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@@
+      (effects (font (size 1.27 1.27)) hide)
+    )
+    (property "JLCPCB Part #" "C116677" (at 38.1 64.77 0)
+      (effects (font (size 1.27 1.27)) hide)
+    )
+    (property "LCSC Part" "C116677" (at 38.1 64.77 0)
       (effects (font (size 1.27 1.27)) hide)
     )
@@
       (effects (font (size 1.27 1.27)) hide)
     )
-    (property "JLCPCB Part #" "" (at 38.1 74.93 0)
+    (property "JLCPCB Part #" "C105907" (at 38.1 74.93 0)
+      (effects (font (size 1.27 1.27)) hide)
+    )
+    (property "LCSC Part" "C105907" (at 38.1 74.93 0)
       (effects (font (size 1.27 1.27)) hide)
     )
@@
   )
   (symbol (lib_id "EduboardV2_kicadlib:EduboardUPConnector_V1") (at 218.44 39.37 0) (unit 1)
-    (in_bom yes) (on_board yes) (dnp no) (fields_autoplaced)
+    (in_bom no) (on_board yes) (dnp no) (fields_autoplaced)
     (property "Reference" "J1" (at 224.79 34.29 0)
       (effects (font (size 1.27 1.27)))
@@
       (effects (font (size 1.27 1.27)) hide)
     )
+    (property "JLCPCB Part #" "C116677" (at 113.665 129.54 0)
+      (effects (font (size 1.27 1.27)) hide)
+    )
+    (property "LCSC Part" "C116677" (at 113.665 129.54 0)
+      (effects (font (size 1.27 1.27)) hide)
+    )
     (pin "1")
     (pin "2")
@@
       (effects (font (size 1.27 1.27)) hide)
     )
+    (property "JLCPCB Part #" "C116677" (at 116.205 129.54 0)
+      (effects (font (size 1.27 1.27)) hide)
+    )
+    (property "LCSC Part" "C116677" (at 116.205 129.54 0)
+      (effects (font (size 1.27 1.27)) hide)
+    )
     (pin "1")
     (pin "2")
@@
       (effects (font (size 1.27 1.27)) hide)
     )
+    (property "JLCPCB Part #" "C115003" (at 44.45 59.69 0)
+      (effects (font (size 1.27 1.27)) hide)
+    )
+    (property "LCSC Part" "C115003" (at 44.45 59.69 0)
+      (effects (font (size 1.27 1.27)) hide)
+    )
     (pin "1")
     (pin "2")
@@
     )
     (property "Datasheet" "~" (at 38.1 34.29 0)
+      (effects (font (size 1.27 1.27)) hide)
+    )
+    (property "JLCPCB Part #" "C116677" (at 38.1 34.29 0)
+      (effects (font (size 1.27 1.27)) hide)
+    )
+    (property "LCSC Part" "C116677" (at 38.1 34.29 0)
       (effects (font (size 1.27 1.27)) hide)
     )
@@
       (effects (font (size 1.27 1.27)) hide)
     )
-    (property "JLCPCB Part #" "" (at 66.04 105.41 0)
+    (property "JLCPCB Part #" "C128624" (at 66.04 105.41 0)
+      (effects (font (size 1.27 1.27)) hide)
+    )
+    (property "LCSC Part" "C128624" (at 66.04 105.41 0)
       (effects (font (size 1.27 1.27)) hide)
     )
@@
       (effects (font (size 1.27 1.27)) hide)
     )
-    (property "JLCPCB Part #" "" (at 76.2 105.41 0)
+    (property "JLCPCB Part #" "C105907" (at 76.2 105.41 0)
+      (effects (font (size 1.27 1.27)) hide)
+    )
+    (property "LCSC Part" "C105907" (at 76.2 105.41 0)
       (effects (font (size 1.27 1.27)) hide)
     )
@@
   )
   (symbol (lib_id "Jumper:SolderJumper_3_Bridged12") (at 179.07 52.07 0) (mirror y) (unit 1)
-    (in_bom yes) (on_board yes) (dnp no)
+    (in_bom no) (on_board yes) (dnp no)
     (property "Reference" "JP8" (at 175.895 53.34 0)
       (effects (font (size 1.27 1.27)))
@@
       (effects (font (size 1.27 1.27)) hide)
     )
+    (property "JLCPCB Part #" "C116677" (at 147.32 131.445 0)
+      (effects (font (size 1.27 1.27)) hide)
+    )
+    (property "LCSC Part" "C116677" (at 147.32 131.445 0)
+      (effects (font (size 1.27 1.27)) hide)
+    )
     (pin "1")
     (pin "2")
@@
   )
   (symbol (lib_id "Jumper:SolderJumper_3_Bridged12") (at 179.07 49.53 180) (unit 1)
-    (in_bom yes) (on_board yes) (dnp no)
+    (in_bom no) (on_board yes) (dnp no)
     (property "Reference" "JP7" (at 175.895 48.26 0)
       (effects (font (size 1.27 1.27)))
@@
       (effects (font (size 1.27 1.27)) hide)
     )
-    (property "JLCPCB Part #" "" (at 38.1 44.45 0)
-      (effects (font (size 1.27 1.27)) hide)
-    )
+    (property "JLCPCB Part #" "C105907" (at 38.1 44.45 0)
+      (effects (font (size 1.27 1.27)) hide)
+    )
+    (property "LCSC Part" "C105907" (at 38.1 44.45 0)
+      (effects (font (size 1.27 1.27)) hide)
+    )
